File: Eagle/QuackDrive/QuackDrive.brd (EAGLE design)
At the start: 160 x 100 mm, 64 parts, among them IC1 MCP1703T-3302E/CB, IC10 TB67H450FNG,EL, IC12 TB67H450FNG,EL, IC2 MCP1703T-3302E/CB, IC4 TB67H450FNG,EL, IC5 ACS70331EOLCTR-2P5U3, IC6 TB67H450FNG,EL, IC8 TB67H450FNG,EL, Q1 NPN-BJT, Q2 NPN-BJT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

Commit message: Liad out motor drives
Parts:
- removed PAD4, PAD7, VBAT: (no value), wirepad:SMD2,54-5,08
- added GND, VBAT_IN: (no value), wirepad:SMD2,54-5,08
- added PAD3: WIREPADSMD1,27-254, wirepad:SMD1,27-2,54
- PAD1, PAD10, PAD11, PAD12, PAD2, PAD5, PAD6, PAD8, PAD9: value (none) -> WIREPADSMD1,27-254; device wirepad:SMD2,54-5,08 -> wirepad:SMD1,27-2,54
- moved UC1 70.9 mm to (26.7, 67.2), turned to 225 degrees
- moved U1 55.1 mm to (42.3, 52.1)
- moved PAD1 54.8 mm to (9.60, 52.1), turned to 90 degrees
- moved IC12 53.8 mm to (14.5, 59.5), turned to 180 degrees
- moved IC4 50.8 mm to (14.5, 70.5), turned to 180 degrees
- moved PAD11 49.5 mm to (9.60, 63.1), turned to 90 degrees
- moved PAD2 49.2 mm to (9.60, 54.7), turned to 270 degrees
- moved PAD12 48.3 mm to (9.60, 65.7), turned to 270 degrees
- moved PAD9 44.9 mm to (9.60, 68.6), turned to 270 degrees
- moved PAD8 39.8 mm to (9.60, 49.1), turned to 90 degrees
- moved PAD6 37.8 mm to (9.60, 60.2), turned to 90 degrees
- moved IC5 36.7 mm to (14.5, 54.0), flipped to the bottom, turned to 180 degrees
- moved PAD5 34.7 mm to (9.60, 57.6), turned to 90 degrees
- moved IC10 32.6 mm to (14.5, 48.5), turned to 180 degrees
- moved IC8 32.2 mm to (14.5, 54.0), turned to 180 degrees
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Connections:
- removed net N$12: IC5.1, IC5.2, VBAT.1
- removed net N$25: IC12.6, PAD12.1
- removed net N$26: IC12.8, PAD11.1
- removed net N$27: IC5.3, IC5.4
- new net N$14: IC8.6, PAD2.1
- new net N$18: IC10.8, PAD3.1
- new net N$21: IC4.6, PAD10.1
- new net VBAT_CUR: IC10.5, IC12.5, IC4.5, IC5.3, IC5.4, IC6.5, IC8.5
- new net VBAT_IN: IC5.1, IC5.2, VBAT_IN.1
- net DGND: now also GND.1, IC10.9, IC12.9, IC4.9, IC6.9, IC8.9; no longer IC10.7, IC12.7, IC4.7, IC6.7, IC8.7, PAD4.1
- net N$11: now also IC12.8, PAD5.1; no longer IC4.6, PAD2.1
- net N$13: now also IC12.6, PAD6.1; no longer IC4.8, PAD1.1
- net N$15: now also IC8.8, PAD1.1; no longer IC6.6, PAD6.1
- net N$17: now also IC10.6, PAD8.1; no longer IC6.8, PAD5.1
- net N$19: now also IC6.6, PAD12.1; no longer IC8.6, PAD8.1
- net N$20: now also IC6.8, PAD11.1; no longer IC8.8, PAD7.1
- net N$22: now also IC4.8, PAD9.1; no longer IC10.6, PAD10.1
- net N$23: now also IC6.4; no longer IC10.8, PAD9.1
- net VCC: no longer IC10.4, IC12.4, IC4.4, IC6.4, IC8.4
Routing:
- net DGND: track 0.00 -> 47.8 mm, vias 0 -> 2
- net VBAT_CUR: track 0.00 -> 44.8 mm, vias 0 -> 4
- net N$17: track 0.00 -> 2.22 mm
- net N$18: track 0.00 -> 2.20 mm
- net N$15: track 0.00 -> 2.19 mm
- net N$19: track 0.00 -> 2.19 mm
- net N$11: track 0.00 -> 2.19 mm
- net N$21: track 0.00 -> 2.19 mm
- net N$22: track 0.00 -> 2.19 mm
- net N$20: track 0.00 -> 2.19 mm
- net N$14: track 0.00 -> 2.19 mm
- net N$13: track 0.00 -> 2.19 mm
- net VBAT_IN: track 0.00 -> 1.27 mm
Other:
- outline, holes or cut-outs redrawn

Commit message: More layout
Parts:
- added R15, R16, R17, R18, R19: .175, SparkFun:C0402
- moved VBAT_IN 46.0 mm to (10.8, 48.5), flipped to the bottom
- moved GND 36.1 mm to (16.6, 70.2), flipped to the bottom
- moved UC1 0.11 mm to (26.6, 67.2)
Connections:
- removed net VDD: IC5.8
- new net N$12: IC6.7, R16.2
- new net N$24: IC8.7, R18.2
- new net N$25: IC12.7, R19.2
- new net N$26: IC4.7, R15.2
- net DGND: now also R15.1, R16.1, R17.1, R18.1, R19.1
- net N$23: now also IC10.7, R17.2; no longer IC6.4
- net VCC: now also IC10.4, IC12.4, IC4.4, IC5.8, IC6.4, IC8.4
Routing:
- net DGND: track 47.8 -> 78.5 mm, vias 2 -> 7
- net VCC: track 0.00 -> 29.4 mm, vias 0 -> 1
- net N$12: track 0.00 -> 1.29 mm
- net N$26: track 0.00 -> 1.29 mm
- net N$23: track 0.00 -> 1.29 mm
- net N$25: track 0.00 -> 1.29 mm
- net N$24: track 0.00 -> 1.29 mm
- net VBAT_CUR: vias 4 -> 3

Commit message: 3d stuff
Other:
- board size 160 x 100 mm -> 12 x 29 mm
