File: Eagle/QuackDrive/QuackDrive.brd (EAGLE design)
At the start: 12 x 29 mm, 69 parts, among them IC1 MCP1703T-3302E/CB, IC10 TB67H450FNG,EL, IC12 TB67H450FNG,EL, IC2 MCP1703T-3302E/CB, IC4 TB67H450FNG,EL, IC5 ACS70331EOLCTR-2P5U3, IC6 TB67H450FNG,EL, IC8 TB67H450FNG,EL, Q1 NPN-BJT, Q2 NPN-BJT, U1 MPU-6050-1, U4 AS5600, X1 USB-MINIB

Commit message: routed power board
Parts:
- removed GND: (no value), wirepad:SMD2,54-5,08
- added PAD4, PAD7: (no value), wirepad:SMD1,27-2,54
- added PWR_GND, PWR_GND1: (no value), wirepad:SMD2,54-5,08
- added R22: 500, SparkFun:C0402
- added R23: 1000, SparkFun:C0402
- added U$1: WM8952DKR, WM8952DKR:SOP80P420X355-16N
- moved UC1 16.0 mm to (42.6, 66.3)
- moved SJ4 0.45 mm to (93.1, 66.5)
- moved VBAT_IN 0.38 mm to (10.5, 48.7), turned to 180 degrees
Connections:
- removed net 27_MOT4_IN1: IC10.2, UC1.29
- removed net 28_MOT4_IN2: IC10.3, UC1.28
- removed net 7_CUR: IC5.7, UC1.14
- removed net DGND: C1.C, C10.1, C11.1, C12.1, C13.1, C14.1, C2.2, C5.2, C6.2, C7.2, C8.2, C9.2, D1.C, GND.1, IC1.1, IC10.1, IC10.9, IC12.1, IC12.9, IC4.1, IC4.9, IC5.5, IC6.1, IC6.9, IC8.1, IC8.9, L1.2, Q1.2, R11.1, R15.1, R16.1, R17.1, R18.1, R19.1, R4.1, R9.1, U1.18, U4.4, UC1.23, UC1.35, UC1.47, X1.GND
- new net 19: UC1.39
- new net 20: UC1.38
- new net 23: UC1.33
- new net 24: UC1.32
- new net 27: UC1.29
- new net 28: UC1.28
- new net 29: UC1.27
- new net 3: UC1.18
- new net 30: UC1.26
- new net 4: UC1.17
- new net 5: UC1.16
- new net 7: UC1.14
- new net 8: UC1.13
- new net N$27: IC5.7, U$1.16
- new net N$28: IC10.2, U$1.4
- new net N$30: R23.1
- new net N$31: IC10.3, U$1.3
- new net N$32: R22.2
- new net N$33: R22.1, R23.2
- new net PWR_GND: IC10.1, IC10.9, IC12.1, IC12.9, IC4.1, IC4.9, IC5.5, IC6.1, IC6.9, IC8.1, IC8.9, PWR_GND.1, R15.1, R16.1, R17.1, R18.1, R19.1, U$1.12, U$1.13
- new net PWR_VCC: IC10.4, IC12.4, IC4.4, IC5.8, IC6.4, IC8.4, U$1.14, U$1.15
- net 19_MOT5_IN1: now also U$1.5; no longer UC1.39
- net 20_MOT5_IN2: now also U$1.6; no longer UC1.38
- net 23_USBDP: no longer UC1.33
- net 24_USBDM: no longer UC1.32
- net 29_MOT3_IN1: now also U$1.2; no longer UC1.27
- net 30_MOT3_IN2: now also U$1.1; no longer UC1.26
- net 3_MOT1_IN1: now also U$1.9; no longer UC1.18
- net 4_MOT1_IN2: now also U$1.8; no longer UC1.17
- net 5_MOT2_IN1: now also U$1.11; no longer UC1.16
- net 8_MOT2_IN2: now also U$1.10; no longer UC1.13
- net GND: now also C1.C, C10.1, C11.1, C12.1, C13.1, C14.1, C2.2, C5.2, C6.2, C7.2, C8.2, C9.2, D1.C, IC1.1, L1.2, Q1.2, R11.1, R4.1, R9.1, U1.18, U4.4, UC1.23, UC1.35, UC1.47, X1.GND
- net VBAT_CUR: now also U$1.7
- net VCC: no longer IC10.4, IC12.4, IC4.4, IC5.8, IC6.4, IC8.4
Routing:
- net PWR_GND: track 0.00 -> 83.0 mm, vias 0 -> 13
- net DGND: track 78.5 -> 0.00 mm, vias 7 -> 0
- net PWR_VCC: track 0.00 -> 35.3 mm, vias 0 -> 2
- net VCC: track 29.4 -> 0.00 mm, vias 1 -> 0
- net 4_MOT1_IN2: track 0.00 -> 20.2 mm, vias 0 -> 1
- net 3_MOT1_IN1: track 0.00 -> 13.8 mm, vias 0 -> 1
- net N$27: track 0.00 -> 13.1 mm
- net N$28: track 0.00 -> 12.5 mm, vias 0 -> 1
- net N$31: track 0.00 -> 10.6 mm, vias 0 -> 1
- net 8_MOT2_IN2: track 0.00 -> 9.70 mm, vias 0 -> 1
- net 29_MOT3_IN1: track 0.00 -> 7.76 mm, vias 0 -> 1
- net 5_MOT2_IN1: track 0.00 -> 7.63 mm, vias 0 -> 1
- net 20_MOT5_IN2: track 0.00 -> 6.14 mm, vias 0 -> 1
- net VBAT_IN: track 1.27 -> 6.82 mm
- net 19_MOT5_IN1: track 0.00 -> 5.15 mm, vias 0 -> 1
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Other:
- board size 12 x 29 mm -> 11.6 x 27.8 mm
