File: Eagle/QuackDrive/QuackDrive.brd (EAGLE design)
At the start: 11.6 x 27.8 mm, 75 parts, among them IC1 MCP1703T-3302E/CB, IC10 TB67H450FNG,EL, IC12 TB67H450FNG,EL, IC2 MCP1703T-3302E/CB, IC4 TB67H450FNG,EL, IC5 ACS70331EOLCTR-2P5U3, IC6 TB67H450FNG,EL, IC8 TB67H450FNG,EL, Q1 NPN-BJT, Q2 NPN-BJT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

Commit message: Maybe finished routing
Parts:
- removed JP1: DNP, Discrete-new:3P-SMD
- removed PWR_GND, PWR_GND1, VBAT_IN: (no value), wirepad:SMD2,54-5,08
- removed R20: 4.7k, Discrete-new:R0402
- removed X1: USB-MINIB, SparkFun2:USB-MINIB
- added C15: 100nf, SparkFun:C0402
- added GND: (no value), wirepad:SMD2,54-5,08
- added PAD13, PAD14, PAD15, PAD16, PAD17, PAD18, PAD19, PAD20: (no value), wirepad:SMD1,27-2,54
- added U$2: SSWTCH, Safet switch:SSWITCH
- added U$3: WM8952DKR, WM8952DKR FW:SOP80P420X355-16N
- added U$4: SSWTCH, Safet switch other side:SSWITCH
- moved R13 94.5 mm to (21.6, 47.2), turned to 270 degrees
- moved R12 90.3 mm to (27.6, 52.8), flipped to the bottom, turned to 180 degrees
- moved R14 90.0 mm to (22.7, 47.3), turned to 270 degrees
- moved R2 89.5 mm to (21.2, 59.9), flipped to the bottom, turned to 90 degrees
- moved D1 89.2 mm to (23.0, 66.2), flipped to the bottom
- moved SJ3 88.4 mm to (30.3, 47.0), turned to 90 degrees
- moved R1 88.0 mm to (24.9, 68.0), flipped to the bottom, turned to 180 degrees
- moved U4 85.9 mm to (1.78, 66.7), turned to 270 degrees
- moved C6 83.6 mm to (23.9, 47.2), turned to 270 degrees
- moved IC1 81.7 mm to (22.6, 68.2), turned to 270 degrees
- moved D2 79.4 mm to (23.5, 64.6), flipped to the bottom
- moved R5 79.4 mm to (21.3, 56.5), turned to 270 degrees
- moved C4 78.8 mm to (31.1, 67.7), turned to 270 degrees
- moved R4 78.3 mm to (26.8, 55.1), turned to 180 degrees
- moved R3 77.4 mm to (30.9, 56.7), turned to 270 degrees
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Connections:
- net 19_MOT5_IN1 renamed MOT5_IN1
- net 20_MOT5_IN2 renamed MOT5_IN2
- net 29_MOT3_IN1 renamed MOT3_IN1
- net 30_MOT3_IN2 renamed MOT3_IN2
- net 3_MOT1_IN1 renamed MOT1_IN1
- net 4_MOT1_IN2 renamed MOT1_IN2
- net 5_MOT2_IN1 renamed MOT2_IN1
- net 8_MOT2_IN2 renamed MOT2_IN2
- net N$27 renamed VIOUT
- net N$28 renamed MOT4_IN1
- net N$31 renamed MOT4_IN2
- removed net 3V3: R20.2, U4.2
- removed net N$30: R23.1
- removed net N$32: R22.2
- removed net N$33: R22.1, R23.2
- removed net VBAT: UC1.1
- net +5V/2: now also PAD18.1; no longer X1.VBUS
- net 10: now also U$3.8
- net 24: now also U$3.1
- net 25: now also U$3.2
- net 26: now also U$3.3
- net 27: now also U$3.4
- net 28: now also U$3.5
- net 29: now also U$3.6
- net 3: now also PAD14.1, U$3.11
- net 4: now also U$3.10
- net 5: now also U$3.9
- net 6: now also U$3.16
- net 7: now also R22.1, R23.2
- net GND: now also PAD15.1, PAD17.1, R23.1, U$3.12, U$3.13; no longer JP1.00, U4.4, X1.GND
- net N$10: now also PAD13.1, U4.3; no longer JP1.MM, U4.8
- net N$16: now also C15.1, PAD7.1, U4.1, U4.2; no longer JP1.11, R20.1
- net N$29: now also C15.2, U4.4, U4.8; no longer PAD7.1
- net N$59: now also PAD19.1; no longer X1.D-
- net N$60: now also PAD20.1; no longer X1.D+
- net PWR_GND: now also GND.1; no longer PWR_GND.1
- net VBAT_IN: now also U$2.SSWTCH_+; no longer VBAT_IN.1
- net VCC: now also PAD16.1, U$3.14, U$3.15, UC1.1; no longer U4.1
- net VIN: now also R22.2, U$3.7
Routing:
- net GND: track 0.00 -> 108.5 mm, vias 0 -> 14
- net VCC: track 0.00 -> 82.6 mm, vias 0 -> 7
- net VBAT_CUR: track 47.7 -> 80.4 mm, vias 3 -> 20
- net N$71: track 0.00 -> 31.8 mm, vias 0 -> 5
- net VIN: track 0.00 -> 28.1 mm, vias 0 -> 5
- net 7: track 0.00 -> 16.5 mm, vias 0 -> 1
- net AV+: track 0.00 -> 16.4 mm, vias 0 -> 2
- net AV-: track 0.00 -> 15.4 mm, vias 0 -> 3
- net N$16: track 0.00 -> 15.3 mm, vias 0 -> 1
- net N$8: track 0.00 -> 15.1 mm, vias 0 -> 2
- net N$29: track 2.21 -> 15.7 mm, vias 0 -> 1
- net OSC_IN: track 0.00 -> 12.1 mm, vias 0 -> 1
- net 29: track 0.00 -> 11.7 mm, vias 0 -> 1
- net OSC_OUT: track 0.00 -> 11.5 mm
- net 28: track 0.00 -> 11.3 mm, vias 0 -> 1
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- added copper zone on layer 16, net GND
- added copper zone on layer 16, net PWR_GND
- added copper zone on layer 1, net VBAT_CUR
- added copper zone on layer 16, net VBAT_CUR
Other:
- board size 11.6 x 27.8 mm -> 24.8 x 27.8 mm

Commit message: stuff
Parts:
- added C16, C19: 10uF, SparkFun:EIA3216
- added C17: .1uF, SparkFun:C0402
- added D3, D4: Blue, SparkFun:LED-1206
- added LED1: Red, Testing:0603-LED-ALT1
- added PAD21, PAD22, PAD24: (no value), wirepad:SMD1,27-2,54
- added R20: 10k, SparkFun:C0402
- added R21, R24: 1k, SparkFun:C0402
- added SJ5, SJ6, SJ7, SJ8: SOLDERJUMPERNO, SparkFun:SJ_2S-NO
- added U$5: WM8952DKR, WM8952DKR:SOP80P420X355-16N
- added U$6: WM8952DKR, WM8952DKR other half:SOP80P420X355-16N
- added U$7: WM8952DKR, WM8952DKR F:SOP80P420X355-16N
- added U$8: WM8952DKR, WM8952DKR F other half:SOP80P420X355-16N
- added U2: MIC5205, SparkFun:SOT23-5
- SJ1, SJ2, SJ3, SJ4: value (none) -> SOLDERJUMPERNO; device SparkFun:SJ_2S-TRACE -> SparkFun:SJ_2S-NO
- moved PAD13 47.6 mm to (4.11, 23.6)
- moved PAD4 47.6 mm to (5.90, 23.6)
- moved PAD7 47.6 mm to (7.72, 23.6)
- moved U4 46.0 mm to (5.90, 21.0)
- moved C9 44.7 mm to (34.8, 16.6)
- moved PAD14 44.2 mm to (34.9, 25.3)
- moved C3 44.2 mm to (33.3, 22.5)
- moved PAD16 44.2 mm to (34.9, 26.7)
- moved PAD6 44.2 mm to (14.4, 16.3)
- moved R2 44.2 mm to (26.2, 16.0)
- moved R23 44.2 mm to (32.8, 27.5)
- moved C10 44.1 mm to (29.1, 27.7)
- moved PAD18 44.1 mm to (27.2, 28.0)
- moved PAD9 44.1 mm to (14.4, 24.7)
- moved R15 44.1 mm to (14.6, 26.0)
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Connections:
- net N$10 renamed MAG_OUT
- new net 5V: C16.A, C17.2, LED1.A, PAD21.1, U2.5
- new net MAG_GND: C15.2, D3.C, D4.C, PAD4.1, SJ7.2, U4.4
- new net MAG_PWR: C15.1, PAD7.1, R21.2, R24.2, SJ8.1, U4.1, U4.2
- new net N$28: D3.A, R21.1
- new net N$30: LED1.C, R20.2
- new net N$32: D4.A, R24.1
- new net N$33: U$7.1, U$8.1
- new net N$34: U$5.2, U$6.2
- new net N$35: U$5.3, U$6.3
- new net N$36: U$5.4, U$6.4
- new net N$37: U$5.5, U$6.5
- new net N$38: U$5.6, U$6.6
- new net N$39: U$5.7, U$6.7
- new net N$40: U$5.8, U$6.8
- new net N$41: U$5.9, U$6.9
- new net N$42: U$5.10, U$6.10
- new net N$43: U$5.11, U$6.11
- new net N$44: U$5.12, U$6.12
- new net N$45: U$5.13, U$6.13
- new net N$46: U$5.14, U$6.14
- new net N$47: U$5.15, U$6.15
- new net N$48: U$5.16, U$6.16
- new net N$49: U$7.2, U$8.2
- new net N$50: U$7.3, U$8.3
- new net N$52: U$7.4, U$8.4
- new net N$53: U$7.5, U$8.5
- new net N$54: U$7.6, U$8.6
- new net N$55: U$7.7, U$8.7
- new net N$56: U$7.8, U$8.8
- new net N$57: U$7.9, U$8.9
- new net N$58: U$7.10, U$8.10
- new net N$6: SJ5.2, U$2.SSWTCH_-
- new net N$61: U$7.11, U$8.11
- new net N$62: U$7.12, U$8.12
- new net N$63: U$7.13, U$8.13
- new net N$64: U$7.14, U$8.14
- new net N$65: U$7.15, U$8.15
- new net N$66: U$7.16, U$8.16
- net 8: now also PAD24.1
- net N$16: now also U$5.1, U$6.1; no longer C15.1, PAD7.1, U4.1, U4.2
- net N$29: now also SJ7.1, SJ8.2; no longer C15.2, PAD4.1, U4.4
- net PWR_GND: now also C16.C, C17.1, C19.C, PAD22.1, R20.1, U2.2
- net VBAT_CUR: now also C19.A, SJ5.1, SJ6.1, SJ6.2, U2.1, U2.3
Routing:
- net VBAT_CUR: track 80.4 -> 121.4 mm, vias 20 -> 22
- net PWR_GND: track 84.6 -> 125.4 mm, vias 41 -> 34
- net MAG_PWR: track 0.00 -> 22.9 mm, vias 0 -> 3
- net MAG_GND: track 0.00 -> 19.0 mm, vias 0 -> 4
- net N$16: track 15.3 -> 0.90 mm, vias 1 -> 2
- net 5V: track 0.00 -> 12.8 mm
- net 8: track 0.00 -> 9.99 mm, vias 0 -> 1
- net N$29: track 15.7 -> 5.86 mm
- net N$30: track 0.00 -> 7.03 mm
- net GND: track 108.5 -> 103.3 mm
- net MOT1_IN1: track 13.5 -> 18.0 mm
- net MOT1_IN2: track 18.7 -> 22.7 mm
- net N$6: track 0.00 -> 3.90 mm
- net N$45: track 0.00 -> 3.21 mm, vias 0 -> 2
- net MAG_OUT: track 6.76 -> 3.69 mm
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- removed copper zone on layer 16, net VBAT_CUR
Other:
- board size 24.8 x 27.8 mm -> 35.9 x 27.9 mm
- board text added: "+"
- board text added: "-"
- board text added: "3v"
- board text added: "5 Pixies"
- board text added: "Allways On"
- board text added: "CLKIN"
- board text added: "Der-M"
- board text added: "Der-P"
- board text added: "FSYNC"
- board text added: "G+-5"
- board text added: "GROUNDDDD"
- board text added: "Gnd"
- board text added: "IDK?"
- board text added: "Live Mount"
- board text added: "Out"
- board text added: "Quack 1"
- board text added: "Quack 2"
- board text added: "Quack 3"
- board text added: "Quack 4"
- board text added: "Quack 5"
- board text added: "RST"
- board text added: "S3G"
- board text added: "Smol Gnd"
- board text added: "Sometimes On"
- board text added: "Warrenty Viod if visible"
- board text added: "You spin me right round"
- board text added: "lol jks, no warrent to start with"

Commit message: Pictures and fixxes
Parts:
- removed IC5: ACS70331EOLCTR-2P5U3, ACS70331EOLCTR-2P5U3:SOIC127P600X175-8N
- removed PAD24: (no value), wirepad:SMD1,27-2,54
- removed R4: 1k, SparkFun:C0402
- added PAD23: (no value), wirepad:SMD1,27-2,54
- added U3: ACS70331EESATR-005B3, ACS70331EESATR-005B3:XDCR_ACS70331EESATR-005B3
- R13, R14: value 10k -> 2k
- moved R5 0.58 mm to (26.5, 12.2)
- moved U1 0.49 mm to (29.5, 7.47)
- moved OSC 0.45 mm to (34.7, 7.33)
- moved R3 0.34 mm to (35.0, 13.2)
- moved C9 0.28 mm to (34.9, 16.8)
- moved L1 0.21 mm to (35.5, 19.8)
- moved R14 0.16 mm to (27.5, 3.22)
- moved C6 0.15 mm to (28.7, 3.22)
- moved R13 0.15 mm to (26.4, 3.22)
- moved SJ2 0.14 mm to (30.0, 3.04)
- moved SJ4 0.12 mm to (31.2, 12.6)
- moved C12 0.09 mm to (31.3, 3.22)
- moved C13 0.08 mm to (33.5, 3.22)
- moved C14 0.07 mm to (32.4, 3.22)
- moved SJ1 0.05 mm to (26.6, 14.5)
Connections:
- removed net N$3: R13.1, U1.23
- removed net N$4: R4.2, SJ4.2
- removed net N$5: R14.1, U1.24
- net 0: now also R13.1, U1.23
- net 1: now also R14.1, U1.24
- net 11: now also U$3.7
- net 15: now also U$3.5
- net 16: now also U$3.1
- net 24: no longer U$3.1
- net 28: no longer U$3.5
- net 29: no longer U$3.6
- net 8: now also PAD23.1; no longer PAD24.1
- net GND: now also SJ4.2; no longer R4.1
- net MOT5_IN2: now also U$1.7; no longer U$1.6
- net PWR_GND: now also U3.5; no longer IC5.5
- net PWR_VCC: now also U3.12; no longer IC5.8
- net VBAT_CUR: now also U$1.6, U3.3_4; no longer IC5.3, IC5.4, U$1.7
- net VBAT_IN: now also U3.1_2; no longer IC5.1, IC5.2
- net VIN: now also U$3.6; no longer U$3.7
- net VIOUT: now also U3.10; no longer IC5.7
Routing:
- net 1: track 0.00 -> 31.1 mm, vias 0 -> 4
- net 0: track 0.00 -> 28.4 mm, vias 0 -> 2
- net 29: track 11.7 -> 0.00 mm, vias 1 -> 0
- net 28: track 11.3 -> 0.00 mm, vias 1 -> 0
- net 24: track 9.91 -> 0.00 mm, vias 1 -> 0
- net PWR_GND: track 125.4 -> 133.4 mm
- net VBAT_IN: track 17.7 -> 25.1 mm
- net PWR_VCC: track 33.0 -> 40.3 mm, vias 2 -> 4
- net 11: track 0.00 -> 5.45 mm, vias 0 -> 1
- net GND: track 103.3 -> 97.9 mm, vias 14 -> 15
- net VBAT_CUR: track 121.4 -> 126.1 mm
- net 15: track 0.00 -> 4.12 mm, vias 0 -> 1
- net VCC: track 82.1 -> 86.1 mm, vias 7 -> 10
- net AV-: track 15.4 -> 11.6 mm
- net 16: track 0.00 -> 3.70 mm, vias 0 -> 1
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- removed copper zone on layer 16, net GND
Other:
- board text added: "Ded Mount"
- board text added: "Goose 5"
- board text added: "More Uselesss"
- board text added: "Never gonna give you up Never gonna let you down Never gonna run around and desert you Never gonna make you cry Never gonna say goodbye Never gonna tell a lie and hurt you Never gonna give you up Never gonna let you down Never gonna run around and desert you Never gonna make you cry Never gonna say goodbye Never gonna tell a lie and hurt you"
- board text added: "Right 'round like a record, baby"
- board text added: "Right 'round, 'round, 'round"
- board text added: "SBSUS In"
- board text added: "Spinny Mag"
- board text added: "Uselesss"
- board text added: "UwUSB"
- board text added: "Warranty Viod if visible"
- board text added: "You spin me right 'round, baby"
- board text removed: "Quack 5"
- board text removed: "Warrenty Viod if visible"
- board text removed: "You spin me right round"

Commit message: new reference board desgn
Parts:
- removed C8, C9: 18pF, SparkFun:C0402
- added C18, C20: 18pF, SparkFun-Capacitors:0603
Connections:
- net GND: now also C18.1, C20.1; no longer C8.2, C9.2
- net OSC_IN: now also C20.2; no longer C9.1
- net OSC_OUT: now also C18.2; no longer C8.1
Routing:
- net OSC_OUT: track 11.7 -> 10.0 mm
- net GND: track 97.9 -> 97.1 mm, vias 15 -> 14
Changed lines of the file:
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@@
 <attribute name="VALUE" x="35.833" y="26.9905" size="0.4064" layer="27" rot="R90"/>
-</element>
-<element name="C8" library="SparkFun" package="C0402" value="18pF" x="34.91" y="11.215" smashed="yes" rot="R180">
-<attribute name="VALUE" x="35.9895" y="12.358" size="0.4064" layer="27" rot="R180"/>
-</element>
-<element name="C9" library="SparkFun" package="C0402" value="18pF" x="34.901025" y="16.814884375" smashed="yes" rot="MR90">
-<attribute name="VALUE" x="33.758025" y="15.735384375" size="0.4064" layer="28" rot="MR90"/>
 </element>
 <element name="D1" library="SparkFun" package="LED-1206" value="Blue" x="27.75" y="22.277584375" smashed="yes" rot="MR0">
@@
 <attribute name="PACKAGE" value="WFQFN-12 Allegro MicroSystems LLC" x="17.794921875" y="9.938446875" size="1.778" layer="28" rot="MR180" display="off"/>
 <attribute name="VALUE" x="15.254921875" y="13.748446875" size="1.27" layer="28" rot="MR180"/>
+</element>
+<element name="C18" library="SparkFun-Capacitors" library_urn="urn:adsk.eagle:library:510" package="0603" package3d_urn="urn:adsk.eagle:package:37414/1" value="18pF" x="-5.61310625" y="-3.705925" smashed="yes">
+<attribute name="NAME" x="-5.61310625" y="-2.943925" size="0.6096" layer="25" font="vector" ratio="20" align="bottom-center"/>
+<attribute name="PROD_ID" value="CAP-08267" x="-5.61310625" y="-3.705925" size="1.778" layer="27" display="off"/>
+<attribute name="VALUE" x="-5.61310625" y="-4.467925" size="0.6096" layer="27" font="vector" ratio="20" align="top-center"/>
+</element>
+<element name="C20" library="SparkFun-Capacitors" library_urn="urn:adsk.eagle:library:510" package="0603" package3d_urn="urn:adsk.eagle:package:37414/1" value="18pF" x="-5.61310625" y="-6.9469625" smashed="yes">
+<attribute name="NAME" x="-5.61310625" y="-6.1849625" size="0.6096" layer="25" font="vector" ratio="20" align="bottom-center"/>
+<attribute name="PROD_ID" value="CAP-08267" x="-5.61310625" y="-6.9469625" size="1.778" layer="27" display="off"/>
+<attribute name="VALUE" x="-5.61310625" y="-7.7089625" size="0.6096" layer="27" font="vector" ratio="20" align="top-center"/>
 </element>
 </elements>
@@
 <signal name="OSC_IN">
 <contactref element="UC1" pad="5"/>
-<contactref element="C9" pad="1"/>
 <contactref element="OSC" pad="3"/>
 <wire x1="33.545" y1="9.18" x2="33.6278" y2="9.2628" width="0.2032" layer="1"/>
@@
 <wire x1="33.445871875" y1="15.010465625" x2="32.97621875" y2="15.48011875" width="0.2032" layer="1"/>
 <wire x1="32.97621875" y1="15.48011875" x2="32.97145625" y2="15.48011875" width="0.2032" layer="1"/>
-<wire x1="34.798140625" y1="16.062" x2="34.901025" y2="16.164884375" width="0.2032" layer="16"/>
 <wire x1="34.798140625" y1="16.062" x2="33.5533375" y2="16.062" width="0.2032" layer="16"/>
 <wire x1="32.97145625" y1="15.48011875" x2="33.5533375" y2="16.062" width="0.2032" layer="16"/>
+<contactref element="C20" pad="2"/>
+<wire x1="-4.76310625" y1="-6.9469625" x2="33.545" y2="9.18" width="0" layer="19" extent="1-1"/>
 </signal>
 <signal name="OSC_OUT">
 <contactref element="UC1" pad="6"/>
-<contactref element="C8" pad="1"/>
 <contactref element="OSC" pad="1"/>
-<wire x1="35.6792125" y1="11.215" x2="35.56" y2="11.215" width="0.2032" layer="1"/>
-<wire x1="35.4292125" y1="11.215" x2="35.56" y2="11.215" width="0.2032" layer="1"/>
 <wire x1="34.1578" y1="14.10813125" x2="34.2844" y2="13.98153125" width="0.2032" layer="1"/>
 <wire x1="34.431" y1="11.919" x2="34.856" y2="11.919" width="0.2032" layer="1"/>
 <wire x1="34.2844" y1="12.0656" x2="34.431" y2="11.919" width="0.2032" layer="1"/>
 <wire x1="34.2844" y1="13.98153125" x2="34.2844" y2="12.0656" width="0.2032" layer="1"/>
-<wire x1="34.856" y1="11.919" x2="35.56" y2="11.215" width="0.2032" layer="1"/>
 <wire x1="33.799425" y1="15.36401875" x2="34.1578" y2="15.00564375" width="0.2032" layer="1"/>
 <wire x1="34.1578" y1="15.00564375" x2="34.1578" y2="14.10813125" width="0.2032" layer="1"/>
@@
 <wire x1="35.4" y1="5.925" x2="35.4" y2="7.6157875" width="0.2032" layer="1"/>
 <wire x1="35.4" y1="7.6157875" x2="35.041" y2="7.9747875" width="0.2032" layer="1"/>
-<wire x1="35.56" y1="10.8442125" x2="35.56" y2="11.215" width="0.2032" layer="1"/>
 <wire x1="35.041" y1="10.3252125" x2="35.56" y2="10.8442125" width="0.2032" layer="1"/>
 <wire x1="35.041" y1="7.9747875" x2="35.041" y2="10.3252125" width="0.2032" layer="1"/>
+<contactref element="C18" pad="2"/>
+<wire x1="35.56" y1="10.8442125" x2="34.856" y2="11.919" width="0" layer="19" extent="1-1"/>
+<wire x1="-4.76310625" y1="-3.705925" x2="35.4" y2="5.925" width="0" layer="19" extent="1-1"/>
 </signal>
 <signal name="N$1">
@@
 <contactref element="C10" pad="1"/>
 <contactref element="C11" pad="1"/>
-<contactref element="C8" pad="2"/>
-<contactref element="C9" pad="2"/>
 <contactref element="R11" pad="1"/>
 <contactref element="Q1" pad="2"/>
@@
 <wire x1="31.738209375" y1="10.8754125" x2="31.596821875" y2="10.8754125" width="0.2032" layer="16"/>
 <wire x1="33.718971875" y1="2.805725" x2="33.485" y2="2.571753125" width="0.2032" layer="1"/>
-<via x="34.26" y="11.215" extent="1-16" drill="0.254"/>
 <wire x1="25.66235" y1="22.34765" x2="25.66235" y2="28.92" width="0.2032" layer="16"/>
 <contactref element="U$3" pad="13"/>
@@
 <via x="34.53" y="8.16" extent="1-16" drill="0.254"/>
 <wire x1="34.53" y1="8.16" x2="34.53" y2="10.945" width="0.2032" layer="1"/>
-<wire x1="34.53" y1="10.945" x2="34.26" y2="11.215" width="0.2032" layer="1"/>
 <contactref element="PAD17" pad="1"/>
 <wire x1="27.160046875" y1="23.749953125" x2="27.24" y2="23.67" width="0.2032" layer="16"/>
@@
 <wire x1="32.8453" y1="26.888875" x2="32.8453" y2="26.9777375" width="0.2032" layer="16"/>
 <wire x1="32.8453" y1="26.9777375" x2="34.095940625" y2="28.228378125" width="0.2032" layer="16"/>
-<wire x1="34.901025" y1="17.464884375" x2="34.901025" y2="17.501025" width="0.2032" layer="16"/>
 <wire x1="34.901025" y1="17.501025" x2="35.27" y2="17.87" width="0.2032" layer="16"/>
 <wire x1="35.27" y1="17.87" x2="35.27" y2="18.59975625" width="0.2032" layer="16"/>
@@
 <wire x1="30.140196875" y1="28.31" x2="29.095" y2="28.31" width="0.2032" layer="1"/>
 <wire x1="35.605021875" y1="17.149575" x2="35.2897125" y2="17.464884375" width="0.2032" layer="16"/>
-<wire x1="34.901025" y1="17.464884375" x2="35.2897125" y2="17.464884375" width="0.2032" layer="16"/>
 <wire x1="34.29" y1="11.4009375" x2="35.605021875" y2="12.715959375" width="0.2032" layer="16"/>
 <wire x1="35.605021875" y1="12.715959375" x2="35.605021875" y2="17.149575" width="0.2032" layer="16"/>
@@
 <contactref element="SJ4" pad="2"/>
 <wire x1="30.82176875" y1="12.55754375" x2="30.775703125" y2="12.603609375" width="0.2032" layer="1"/>
-<wire x1="30.4355" y1="12.17" x2="30.775703125" y2="12.603609375" width="0" layer="19" extent="1-16"/>
+<contactref element="C18" pad="1"/>
+<contactref element="C20" pad="1"/>
+<wire x1="35.2897125" y1="17.464884375" x2="34.901025" y2="17.501025" width="0" layer="19" extent="16-16"/>
+<wire x1="34.53" y1="10.945" x2="34.29" y2="11.185" width="0" layer="19" extent="1-16"/>
+<wire x1="30.775703125" y1="12.603609375" x2="30.4355" y2="12.17" width="0" layer="19" extent="1-16"/>
+<wire x1="-6.46310625" y1="-3.705925" x2="26.405" y2="8.74" width="0" layer="19" extent="1-16"/>
+<wire x1="-6.46310625" y1="-6.9469625" x2="-6.46310625" y2="-3.705925" width="0" layer="19" extent="1-1"/>
 </signal>
 <signal name="FSYNC1">

Commit message: Finished off missing bits
Parts:
- moved C20 43.5 mm to (35.4, 7.33), flipped to the bottom, turned to 90 degrees
- moved C18 41.7 mm to (35.3, 4.03), flipped to the bottom, turned to 270 degrees
- moved C4 0.22 mm to (36.1, 24.0)
- moved PAD23 0.21 mm to (35.5, 10.3)
- moved R10 0.09 mm to (30.1, 25.6)
Routing:
- net GND: track 97.1 -> 104.1 mm, vias 14 -> 15
- net OSC_OUT: track 10.0 -> 13.9 mm, vias 0 -> 1
- net OSC_IN: track 8.95 -> 9.59 mm, vias 1 -> 2
