File: Eagle/QuackDrive/QuackDrive.sch (EAGLE design)
At the start: 68 parts, among them IC1 MCP1703T-3302E/CB, IC10 TB67H450FNG,EL, IC11 ACS70331EOLCTR-2P5U3, IC12 TB67H450FNG,EL, IC2 MCP1703T-3302E/CB, IC3 ACS70331EOLCTR-2P5U3, IC4 TB67H450FNG,EL, IC5 ACS70331EOLCTR-2P5U3, IC6 TB67H450FNG,EL, IC7 ACS70331EOLCTR-2P5U3, IC8 TB67H450FNG,EL, IC9 ACS70331EOLCTR-2P5U3, Q1 NPN-BJT, Q2 NPN-BJT, U1 MPU-6050-1, U4 AS5600, X1 USB-MINIB

Commit message: Remove all but one current sens
Parts:
- removed IC11, IC3, IC7, IC9: ACS70331EOLCTR-2P5U3, ACS70331EOLCTR-2P5U3:ACS70331EOLCTR-2P5U3
- removed PAD3: (no value), wirepad:SMD5
- added VBAT: (no value), wirepad:SMD5
Connections:
- net 7_CUR_2 renamed 7_CUR
- removed net 10_CUR_4: IC9.VIOUT, UC1.PA1/USART2_RTS/ADC12_IN1/TIM2_CH2
- removed net 11_CUR_5: IC11.VIOUT, UC1.PA0_WKUP/USART2_CTS/ADC12_IN0/TIM2_CH1_ETR
- removed net 6_CUR_1: IC3.VIOUT, UC1.PA5/SPI1_SCK/ADC12_IN5
- removed net 9_CUR_3: IC7.VIOUT, UC1.PA2/USART2_TX/ADC12_IN2/TIM2_CH3
- removed net N$14: IC5.IP-_1, IC5.IP-_2, IC6.VM
- removed net N$18: IC7.IP-_1, IC7.IP-_2, IC8.VM
- removed net N$21: IC10.VM, IC9.IP-_1, IC9.IP-_2
- removed net N$24: IC11.IP-_1, IC11.IP-_2, IC12.VM
- new net 10: UC1.PA1/USART2_RTS/ADC12_IN1/TIM2_CH2
- new net 11: UC1.PA0_WKUP/USART2_CTS/ADC12_IN0/TIM2_CH1_ETR
- new net 6: UC1.PA5/SPI1_SCK/ADC12_IN5
- new net 9: UC1.PA2/USART2_TX/ADC12_IN2/TIM2_CH3
- new net N$27: IC5.IP-_1, IC5.IP-_2
- net DGND: no longer IC11.GND, IC3.GND, IC7.GND, IC9.GND
- net N$12: now also IC5.IP+_1, IC5.IP+_2, VBAT.P; no longer IC3.IP-_1, IC3.IP-_2, IC4.VM
- net VDD: no longer IC11.IP+_1, IC11.IP+_2, IC11.VCC, IC3.IP+_1, IC3.IP+_2, IC3.VCC, IC5.IP+_1, IC5.IP+_2, IC7.IP+_1, IC7.IP+_2, IC7.VCC, IC9.IP+_1, IC9.IP+_2, IC9.VCC, PAD3.P

Commit message: Liad out motor drives
Parts:
- removed PAD4, PAD7: (no value), wirepad:SMD5
- added GND: (no value), wirepad:SMD5
- added PAD3: WIREPADSMD1,27-254, wirepad:WIREPADSMD1,27-254
- PAD1, PAD10, PAD11, PAD12, PAD2, PAD5, PAD6, PAD8, PAD9: value (none) -> WIREPADSMD1,27-254; device wirepad:SMD5 -> wirepad:WIREPADSMD1,27-254
- renumbered VBAT to VBAT_IN
Connections:
- net N$12 renamed VBAT_IN
- removed net N$25: IC12.OUT1, PAD12.P
- removed net N$26: IC12.OUT2, PAD11.P
- removed net N$27: IC5.IP-_1, IC5.IP-_2
- new net N$14: IC8.OUT1, PAD2.P
- new net N$18: IC10.OUT2, PAD3.P
- new net N$21: IC4.OUT1, PAD10.P
- new net VBAT_CUR: IC10.VM, IC12.VM, IC4.VM, IC5.IP-_1, IC5.IP-_2, IC6.VM, IC8.VM
- net DGND: now also GND.P, IC10.EP, IC12.EP, IC4.EP, IC6.EP, IC8.EP; no longer IC10.RS, IC12.RS, IC4.RS, IC6.RS, IC8.RS, PAD4.P
- net N$11: now also IC12.OUT2, PAD5.P; no longer IC4.OUT1, PAD2.P
- net N$13: now also IC12.OUT1, PAD6.P; no longer IC4.OUT2, PAD1.P
- net N$15: now also IC8.OUT2, PAD1.P; no longer IC6.OUT1, PAD6.P
- net N$17: now also IC10.OUT1, PAD8.P; no longer IC6.OUT2, PAD5.P
- net N$19: now also IC6.OUT1, PAD12.P; no longer IC8.OUT1, PAD8.P
- net N$20: now also IC6.OUT2, PAD11.P; no longer IC8.OUT2, PAD7.P
- net N$22: now also IC4.OUT2, PAD9.P; no longer IC10.OUT1, PAD10.P
- net N$23: now also IC6.VREF; no longer IC10.OUT2, PAD9.P
- net VCC: no longer IC10.VREF, IC12.VREF, IC4.VREF, IC6.VREF, IC8.VREF

Commit message: More layout
Parts:
- added R15, R16, R17, R18, R19: .175, SparkFun:RESISTOR0402
Connections:
- removed net VDD: IC5.VCC
- new net N$12: IC6.RS, R16.2
- new net N$24: IC8.RS, R18.2
- new net N$25: IC12.RS, R19.2
- new net N$26: IC4.RS, R15.2
- net DGND: now also R15.1, R16.1, R17.1, R18.1, R19.1
- net N$23: now also IC10.RS, R17.2; no longer IC6.VREF
- net VCC: now also IC10.VREF, IC12.VREF, IC4.VREF, IC5.VCC, IC6.VREF, IC8.VREF
Changed lines of the file:
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@@
 <?xml version="1.0" encoding="utf-8"?>
 <!DOCTYPE eagle SYSTEM "eagle.dtd">
-<eagle version="9.2.2">
+<eagle version="9.4.2">
 <drawing>
 <settings>
@@
 <part name="SUPPLY44" library="supply2" deviceset="DGND" device="" value="GND"/>
 <part name="SUPPLY47" library="supply2" deviceset="DGND" device="" value="GND"/>
+<part name="P+10" library="SparkFun" deviceset="VCC" device=""/>
+<part name="P+12" library="SparkFun" deviceset="VCC" device=""/>
+<part name="P+13" library="SparkFun" deviceset="VCC" device=""/>
+<part name="P+15" library="SparkFun" deviceset="VCC" device=""/>
+<part name="P+16" library="SparkFun" deviceset="VCC" device=""/>
+<part name="P+17" library="SparkFun" deviceset="VCC" device=""/>
+<part name="R15" library="SparkFun" deviceset="RESISTOR" device="0402" value=".175"/>
+<part name="SUPPLY33" library="supply2" deviceset="DGND" device="" value="GND"/>
+<part name="R16" library="SparkFun" deviceset="RESISTOR" device="0402" value=".175"/>
+<part name="SUPPLY37" library="supply2" deviceset="DGND" device="" value="GND"/>
+<part name="R17" library="SparkFun" deviceset="RESISTOR" device="0402" value=".175"/>
+<part name="SUPPLY40" library="supply2" deviceset="DGND" device="" value="GND"/>
+<part name="R18" library="SparkFun" deviceset="RESISTOR" device="0402" value=".175"/>
+<part name="SUPPLY43" library="supply2" deviceset="DGND" device="" value="GND"/>
+<part name="R19" library="SparkFun" deviceset="RESISTOR" device="0402" value=".175"/>
+<part name="SUPPLY46" library="supply2" deviceset="DGND" device="" value="GND"/>
 </parts>
 <sheets>
@@
 <instance part="SUPPLY47" gate="G$1" x="-154.94" y="207.01" smashed="yes">
 <attribute name="VALUE" x="-157.607" y="203.835" size="1.778" layer="96"/>
+</instance>
+<instance part="P+10" gate="1" x="125.73" y="187.96" smashed="yes" rot="R90">
+<attribute name="VALUE" x="122.174" y="186.944" size="1.778" layer="96" rot="R90"/>
+</instance>
+<instance part="P+12" gate="1" x="-6.35" y="223.52" smashed="yes" rot="R90">
+<attribute name="VALUE" x="-9.906" y="222.504" size="1.778" layer="96" rot="R90"/>
+</instance>
+<instance part="P+13" gate="1" x="-6.35" y="187.96" smashed="yes" rot="R90">
+<attribute name="VALUE" x="-9.906" y="186.944" size="1.778" layer="96" rot="R90"/>
+</instance>
+<instance part="P+15" gate="1" x="-95.25" y="187.96" smashed="yes" rot="R90">
+<attribute name="VALUE" x="-98.806" y="186.944" size="1.778" layer="96" rot="R90"/>
+</instance>
+<instance part="P+16" gate="1" x="-92.71" y="223.52" smashed="yes" rot="R90">
+<attribute name="VALUE" x="-96.266" y="222.504" size="1.778" layer="96" rot="R90"/>
+</instance>
+<instance part="P+17" gate="1" x="-173.99" y="223.52" smashed="yes" rot="R90">
+<attribute name="VALUE" x="-177.546" y="222.504" size="1.778" layer="96" rot="R90"/>
+</instance>
+<instance part="R15" gate="G$1" x="33.02" y="228.6" smashed="yes" rot="R180">
+<attribute name="NAME" x="36.83" y="227.1014" size="1.778" layer="95" rot="R180"/>
+<attribute name="VALUE" x="36.83" y="231.902" size="1.778" layer="96" rot="R180"/>
+</instance>
+<instance part="SUPPLY33" gate="G$1" x="39.37" y="228.6" smashed="yes" rot="R90">
+<attribute name="VALUE" x="42.545" y="225.933" size="1.778" layer="96" rot="R90"/>
+</instance>
+<instance part="R16" gate="G$1" x="31.75" y="194.31" smashed="yes" rot="R180">
+<attribute name="NAME" x="35.56" y="192.8114" size="1.778" layer="95" rot="R180"/>
+<attribute name="VALUE" x="35.56" y="197.612" size="1.778" layer="96" rot="R180"/>
+</instance>
+<instance part="SUPPLY37" gate="G$1" x="40.64" y="194.31" smashed="yes" rot="R90">
+<attribute name="VALUE" x="43.815" y="191.643" size="1.778" layer="96" rot="R90"/>
+</instance>
+<instance part="R17" gate="G$1" x="-55.88" y="194.31" smashed="yes" rot="R180">
+<attribute name="NAME" x="-52.07" y="192.8114" size="1.778" layer="95" rot="R180"/>
+<attribute name="VALUE" x="-52.07" y="197.612" size="1.778" layer="96" rot="R180"/>
+</instance>
+<instance part="SUPPLY40" gate="G$1" x="-46.99" y="194.31" smashed="yes" rot="R90">
+<attribute name="VALUE" x="-43.815" y="191.643" size="1.778" layer="96" rot="R90"/>
+</instance>
+<instance part="R18" gate="G$1" x="-55.88" y="228.6" smashed="yes" rot="R180">
+<attribute name="NAME" x="-52.07" y="227.1014" size="1.778" layer="95" rot="R180"/>
+<attribute name="VALUE" x="-52.07" y="231.902" size="1.778" layer="96" rot="R180"/>
+</instance>
+<instance part="SUPPLY43" gate="G$1" x="-46.99" y="228.6" smashed="yes" rot="R90">
+<attribute name="VALUE" x="-43.815" y="225.933" size="1.778" layer="96" rot="R90"/>
+</instance>
+<instance part="R19" gate="G$1" x="-135.89" y="228.6" smashed="yes" rot="R180">
+<attribute name="NAME" x="-132.08" y="227.1014" size="1.778" layer="95" rot="R180"/>
+<attribute name="VALUE" x="-132.08" y="231.902" size="1.778" layer="96" rot="R180"/>
+</instance>
+<instance part="SUPPLY46" gate="G$1" x="-127" y="228.6" smashed="yes" rot="R90">
+<attribute name="VALUE" x="-123.825" y="225.933" size="1.778" layer="96" rot="R90"/>
 </instance>
 </instances>
@@
 <wire x1="260.35" y1="273.05" x2="261.62" y2="273.05" width="0.1524" layer="91"/>
 </segment>
+<segment>
+<wire x1="128.27" y1="187.96" x2="125.73" y2="187.96" width="0.1524" layer="91"/>
+<pinref part="P+10" gate="1" pin="VCC"/>
+</segment>
+<segment>
+<wire x1="-3.81" y1="223.52" x2="-6.35" y2="223.52" width="0.1524" layer="91"/>
+<pinref part="P+12" gate="1" pin="VCC"/>
+<pinref part="IC4" gate="G$1" pin="VREF"/>
+</segment>
+<segment>
+<pinref part="P+13" gate="1" pin="VCC"/>
+<pinref part="IC6" gate="G$1" pin="VREF"/>
+<wire x1="-5.08" y1="187.96" x2="-6.35" y2="187.96" width="0.1524" layer="91"/>
+<wire x1="-5.08" y1="187.96" x2="-3.81" y2="187.96" width="0.1524" layer="91"/>
+<wire x1="-3.81" y1="187.96" x2="-3.81" y2="189.23" width="0.1524" layer="91"/>
+</segment>
+<segment>
+<wire x1="-92.71" y1="187.96" x2="-93.98" y2="187.96" width="0.1524" layer="91"/>
+<pinref part="P+15" gate="1" pin="VCC"/>
+<pinref part="IC10" gate="G$1" pin="VREF"/>
+<wire x1="-93.98" y1="187.96" x2="-95.25" y2="187.96" width="0.1524" layer="91"/>
+<wire x1="-92.71" y1="187.96" x2="-91.44" y2="187.96" width="0.1524" layer="91"/>
+<wire x1="-91.44" y1="187.96" x2="-91.44" y2="189.23" width="0.1524" layer="91"/>
+</segment>
+<segment>
+<wire x1="-90.17" y1="223.52" x2="-91.44" y2="223.52" width="0.1524" layer="91"/>
+<pinref part="P+16" gate="1" pin="VCC"/>
+<pinref part="IC8" gate="G$1" pin="VREF"/>
+<wire x1="-91.44" y1="223.52" x2="-92.71" y2="223.52" width="0.1524" layer="91"/>
+<junction x="-91.44" y="223.52"/>
+</segment>
+<segment>
+<wire x1="-171.45" y1="223.52" x2="-173.99" y2="223.52" width="0.1524" layer="91"/>
+<pinref part="P+17" gate="1" pin="VCC"/>
+<pinref part="IC12" gate="G$1" pin="VREF"/>
+</segment>
+<segment>
+<pinref part="IC5" gate="G$1" pin="VCC"/>
+<pinref part="VDD7" gate="G$1" pin="VDD"/>
+<wire x1="313.69" y1="113.03" x2="317.5" y2="113.03" width="0.1524" layer="91"/>
+</segment>
 </net>
 <net name="N$51" class="0">
@@
 <wire x1="-76.2" y1="210.82" x2="-74.93" y2="212.09" width="0.1524" layer="91"/>
 <wire x1="-74.93" y1="212.09" x2="-73.66" y2="212.09" width="0.1524" layer="91"/>
+</segment>
+<segment>
+<pinref part="R15" gate="G$1" pin="1"/>
+<pinref part="SUPPLY33" gate="G$1" pin="DGND"/>
+<wire x1="38.1" y1="228.6" x2="36.83" y2="228.6" width="0.1524" layer="91"/>
+</segment>
+<segment>
+<pinref part="R16" gate="G$1" pin="1"/>
+<pinref part="SUPPLY37" gate="G$1" pin="DGND"/>
+<wire x1="36.83" y1="194.31" x2="38.1" y2="194.31" width="0.1524" layer="91"/>
+</segment>
+<segment>
+<pinref part="R17" gate="G$1" pin="1"/>
+<pinref part="SUPPLY40" gate="G$1" pin="DGND"/>
+<wire x1="-50.8" y1="194.31" x2="-49.53" y2="194.31" width="0.1524" layer="91"/>
+</segment>
+<segment>
+<pinref part="R18" gate="G$1" pin="1"/>
+<pinref part="SUPPLY43" gate="G$1" pin="DGND"/>
+<wire x1="-50.8" y1="228.6" x2="-49.53" y2="228.6" width="0.1524" layer="91"/>
+</segment>
+<segment>
+<pinref part="R19" gate="G$1" pin="1"/>
+<pinref part="SUPPLY46" gate="G$1" pin="DGND"/>
+<wire x1="-130.81" y1="228.6" x2="-129.54" y2="228.6" width="0.1524" layer="91"/>
 </segment>
 </net>
@@
 </segment>
 </net>
-<net name="VDD" class="0">
-<segment>
-<pinref part="IC5" gate="G$1" pin="VCC"/>
-<pinref part="VDD7" gate="G$1" pin="VDD"/>
-<wire x1="313.69" y1="113.03" x2="317.5" y2="113.03" width="0.1524" layer="91"/>
-</segment>
-</net>
 <net name="VBAT_CUR" class="0">
 <segment>
@@
 </segment>
 </net>
-<net name="N$23" class="0">
-<segment>
-<pinref part="IC6" gate="G$1" pin="VREF"/>
-<wire x1="-3.81" y1="189.23" x2="-3.81" y2="182.88" width="0.1524" layer="91"/>
-</segment>
-</net>
 <net name="VBAT_IN" class="0">
 <segment>
@@
 </segment>
 </net>
+<net name="N$12" class="0">
+<segment>
+<pinref part="R16" gate="G$1" pin="2"/>
+<pinref part="IC6" gate="G$1" pin="RS"/>
+</segment>
+</net>
+<net name="N$23" class="0">
+<segment>
+<pinref part="R17" gate="G$1" pin="2"/>
+<pinref part="IC10" gate="G$1" pin="RS"/>
+</segment>
+</net>
+<net name="N$24" class="0">
+<segment>
+<pinref part="R18" gate="G$1" pin="2"/>
+<pinref part="IC8" gate="G$1" pin="RS"/>
+</segment>
+</net>
+<net name="N$25" class="0">
+<segment>
+<pinref part="R19" gate="G$1" pin="2"/>
+<pinref part="IC12" gate="G$1" pin="RS"/>
+</segment>
+</net>
+<net name="N$26" class="0">
+<segment>
+<pinref part="R15" gate="G$1" pin="2"/>
+<pinref part="IC4" gate="G$1" pin="RS"/>
+<wire x1="27.94" y1="228.6" x2="26.67" y2="228.6" width="0.1524" layer="91"/>
+</segment>
+</net>

Commit message: routed power board
Parts:
- removed GND: (no value), wirepad:SMD5
- added PAD4, PAD7: (no value), wirepad:SMD2
- added PWR_GND, PWR_GND1: (no value), wirepad:SMD5
- added R22: 500, SparkFun:RESISTOR0402
- added R23: 1000, SparkFun:RESISTOR0402
- added U$1: WM8952DKR, WM8952DKR:WM8952DKR
Connections:
- removed net 27_MOT4_IN1: IC10.IN2, UC1.PA8/USART1_CK/TIM1_CH1/MCO
- removed net 28_MOT4_IN2: IC10.IN1, UC1.PB15/SPI2_MOSI/TIM1_CH3N
- removed net 7_CUR: IC5.VIOUT, UC1.PA4/SPI1_NSS/USART2_CK/ADC12_IN4
- removed net DGND: C1.-, C10.1, C11.1, C12.1, C13.1, C14.1, C2.2, C5.2, C6.2, C7.2, C8.2, C9.2, D1.C, GND.P, IC1.GND, IC10.EP, IC10.GND, IC12.EP, IC12.GND, IC4.EP, IC4.GND, IC5.GND, IC6.EP, IC6.GND, IC8.EP, IC8.GND, L1.2, Q1.E, R11.1, R15.1, R16.1, R17.1, R18.1, R19.1, R4.1, R9.1, U1.GND, U4.GND, UC1.VSS_1, UC1.VSS_2, UC1.VSS_3, X1.GND
- new net 19: UC1.PB3/JTDO
- new net 20: UC1.PA15/JTDI
- new net 23: UC1.PA12/USART1_RTS/CAN_TX/TIM1_ETR/USBDP
- new net 24: UC1.PA11/USART1_CTS/CAN_RX/TIM1_CH4/USBDM
- new net 27: UC1.PA8/USART1_CK/TIM1_CH1/MCO
- new net 28: UC1.PB15/SPI2_MOSI/TIM1_CH3N
- new net 29: UC1.PB14/SPI2_MISO/USART3_RTS/TIM1_CH2N
- new net 3: UC1.PB0/ADC12_IN8/TIM3_CH3
- new net 30: UC1.PB13/SPI2_SCK/USART3_CTS/TIM1_CH1N
- new net 4: UC1.PA7/SPI1_MOSI/ADC12_IN7/TIM3_CH2
- new net 5: UC1.PA6/SPI1_MISO/ADC12_IN6/TIM3_CH1
- new net 7: UC1.PA4/SPI1_NSS/USART2_CK/ADC12_IN4
- new net 8: UC1.PA3/USART2_RX/ADC12_IN3/TIM2_CH4
- new net N$27: IC5.VIOUT, U$1.P$16
- new net N$28: IC10.IN2, U$1.P$4
- new net N$30: R23.1
- new net N$31: IC10.IN1, U$1.P$3
- new net N$32: R22.2
- new net N$33: R22.1, R23.2
- new net PWR_GND: IC10.EP, IC10.GND, IC12.EP, IC12.GND, IC4.EP, IC4.GND, IC5.GND, IC6.EP, IC6.GND, IC8.EP, IC8.GND, PWR_GND.P, R15.1, R16.1, R17.1, R18.1, R19.1, U$1.P$12, U$1.P$13
- new net PWR_VCC: IC10.VREF, IC12.VREF, IC4.VREF, IC5.VCC, IC6.VREF, IC8.VREF, U$1.P$14, U$1.P$15
- net 19_MOT5_IN1: now also U$1.P$5; no longer UC1.PB3/JTDO
- net 20_MOT5_IN2: now also U$1.P$6; no longer UC1.PA15/JTDI
- net 23_USBDP: no longer UC1.PA12/USART1_RTS/CAN_TX/TIM1_ETR/USBDP
- net 24_USBDM: no longer UC1.PA11/USART1_CTS/CAN_RX/TIM1_CH4/USBDM
- net 29_MOT3_IN1: now also U$1.P$2; no longer UC1.PB14/SPI2_MISO/USART3_RTS/TIM1_CH2N
- net 30_MOT3_IN2: now also U$1.P$1; no longer UC1.PB13/SPI2_SCK/USART3_CTS/TIM1_CH1N
- net 3_MOT1_IN1: now also U$1.P$9; no longer UC1.PB0/ADC12_IN8/TIM3_CH3
- net 4_MOT1_IN2: now also U$1.P$8; no longer UC1.PA7/SPI1_MOSI/ADC12_IN7/TIM3_CH2
- net 5_MOT2_IN1: now also U$1.P$11; no longer UC1.PA6/SPI1_MISO/ADC12_IN6/TIM3_CH1
- net 8_MOT2_IN2: now also U$1.P$10; no longer UC1.PA3/USART2_RX/ADC12_IN3/TIM2_CH4
- net GND: now also C1.-, C10.1, C11.1, C12.1, C13.1, C14.1, C2.2, C5.2, C6.2, C7.2, C8.2, C9.2, D1.C, IC1.GND, L1.2, Q1.E, R11.1, R4.1, R9.1, U1.GND, U4.GND, UC1.VSS_1, UC1.VSS_2, UC1.VSS_3, X1.GND
- net VBAT_CUR: now also U$1.P$7
- net VCC: no longer IC10.VREF, IC12.VREF, IC4.VREF, IC5.VCC, IC6.VREF, IC8.VREF
Other:
- moved on the sheet: R15, R16, R17, R18, R19, VBAT_IN

Commit message: ipdate
Connections:
- new net N$29: PAD4.P, PAD7.P
Changed lines of the file:
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@@
 <?xml version="1.0" encoding="utf-8"?>
 <!DOCTYPE eagle SYSTEM "eagle.dtd">
-<eagle version="9.2.2">
+<eagle version="9.4.2">
 <drawing>
 <settings>
@@
 </segment>
 </net>
+<net name="N$29" class="0">
+<segment>
+<pinref part="PAD4" gate="1" pin="P"/>
+<wire x1="5.08" y1="137.16" x2="7.62" y2="137.16" width="0.1524" layer="91"/>
+<wire x1="7.62" y1="137.16" x2="7.62" y2="127" width="0.1524" layer="91"/>
+<pinref part="PAD7" gate="1" pin="P"/>
+<wire x1="7.62" y1="121.92" x2="7.62" y2="127" width="0.1524" layer="91"/>
+<junction x="7.62" y="127"/>
+</segment>
+</net>

Commit message: Maybe finished routing
Parts:
- removed JP1: DNP, Discrete-new:JP-3P
- removed PWR_GND, PWR_GND1, VBAT_IN: (no value), wirepad:SMD5
- removed R20: 4.7k, Discrete-new:RES-0402
- removed X1: USB-MINIB, SparkFun2:USBSMD
- added C15: 100nf, SparkFun:CAP0402
- added GND: (no value), wirepad:SMD5
- added PAD13, PAD14, PAD15, PAD16, PAD17, PAD18, PAD19, PAD20: (no value), wirepad:SMD2
- added U$2: SSWTCH, Safet switch:SSWTCH
- added U$3: WM8952DKR, WM8952DKR FW:WM8952DKR
- added U$4: SSWTCH, Safet switch other side:SSWTCH
Connections:
- net 19_MOT5_IN1 renamed MOT5_IN1
- net 20_MOT5_IN2 renamed MOT5_IN2
- net 29_MOT3_IN1 renamed MOT3_IN1
- net 30_MOT3_IN2 renamed MOT3_IN2
- net 3_MOT1_IN1 renamed MOT1_IN1
- net 4_MOT1_IN2 renamed MOT1_IN2
- net 5_MOT2_IN1 renamed MOT2_IN1
- net 8_MOT2_IN2 renamed MOT2_IN2
- net N$27 renamed VIOUT
- net N$28 renamed MOT4_IN1
- net N$31 renamed MOT4_IN2
- removed net 3V3: R20.2, U4.VDD3V3
- removed net N$30: R23.1
- removed net N$32: R22.2
- removed net N$33: R22.1, R23.2
- removed net VBAT: UC1.VBAT
- net +5V/2: now also PAD18.P; no longer X1.VBUS
- net 10: now also U$3.P$8
- net 24: now also U$3.P$1
- net 25: now also U$3.P$2
- net 26: now also U$3.P$3
- net 27: now also U$3.P$4
- net 28: now also U$3.P$5
- net 29: now also U$3.P$6
- net 3: now also PAD14.P, U$3.P$11
- net 4: now also U$3.P$10
- net 5: now also U$3.P$9
- net 6: now also U$3.P$16
- net 7: now also R22.1, R23.2
- net GND: now also PAD15.P, PAD17.P, R23.1, U$3.P$12, U$3.P$13; no longer JP1.R, U4.GND, X1.GND
- net N$10: now also PAD13.P, U4.OUT; no longer JP1.C, U4.DIR
- net N$16: now also C15.1, PAD7.P, U4.VDD3V3, U4.VDD5V; no longer JP1.L, R20.1
- net N$29: now also C15.2, U4.DIR, U4.GND; no longer PAD7.P
- net N$59: now also PAD19.P; no longer X1.D-
- net N$60: now also PAD20.P; no longer X1.D+
- net PWR_GND: now also GND.P; no longer PWR_GND.P
- net VBAT_IN: now also U$2.P$1; no longer VBAT_IN.P
- net VCC: now also PAD16.P, U$3.P$14, U$3.P$15, UC1.VBAT; no longer U4.VDD5V
- net VIN: now also R22.2, U$3.P$7
Other:
- moved on the sheet: C1, C10, C11, C12, C13, C14, C2, C3, C4, C5, C6, C7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

Commit message: stuff
Parts:
- added C16, C19: 10uF, SparkFun:CAP_POL1206
- added C17: .1uF, SparkFun:CAP0402
- added D3, D4: Blue, SparkFun:LED1206
- added LED1: Red, Testing:LED
- added PAD21, PAD22, PAD24: (no value), wirepad:SMD2
- added R20: 10k, SparkFun:RESISTOR0402
- added R21, R24: 1k, SparkFun:RESISTOR0402
- added SJ5, SJ6, SJ7, SJ8: SOLDERJUMPERNO, SparkFun:SOLDERJUMPERNO
- added U$5: WM8952DKR, WM8952DKR:WM8952DKR
- added U$6: WM8952DKR, WM8952DKR other half:WM8952DKR
- added U$7: WM8952DKR, WM8952DKR F:WM8952DKR
- added U$8: WM8952DKR, WM8952DKR F other half:WM8952DKR
- added U2: MIC5205, SparkFun:V_REG_LDOSMD
- SJ1, SJ2, SJ3, SJ4: value SOLDERJUMPERTRACE -> SOLDERJUMPERNO; device SparkFun:SOLDERJUMPERTRACE -> SparkFun:SOLDERJUMPERNO
Connections:
- net N$10 renamed MAG_OUT
- new net 5V: C16.+, C17.2, LED1.A, PAD21.P, U2.OUT
- new net MAG_GND: C15.2, D3.C, D4.C, PAD4.P, SJ7.2, U4.GND
- new net MAG_PWR: C15.1, PAD7.P, R21.2, R24.2, SJ8.1, U4.VDD3V3, U4.VDD5V
- new net N$28: D3.A, R21.1
- new net N$30: LED1.C, R20.2
- new net N$32: D4.A, R24.1
- new net N$33: U$7.P$1, U$8.P$16
- new net N$34: U$5.P$2, U$6.P$15
- new net N$35: U$5.P$3, U$6.P$14
- new net N$36: U$5.P$4, U$6.P$13
- new net N$37: U$5.P$5, U$6.P$12
- new net N$38: U$5.P$6, U$6.P$11
- new net N$39: U$5.P$7, U$6.P$10
- new net N$40: U$5.P$8, U$6.P$9
- new net N$41: U$5.P$9, U$6.P$8
- new net N$42: U$5.P$10, U$6.P$7
- new net N$43: U$5.P$11, U$6.P$6
- new net N$44: U$5.P$12, U$6.P$5
- new net N$45: U$5.P$13, U$6.P$4
- new net N$46: U$5.P$14, U$6.P$3
- new net N$47: U$5.P$15, U$6.P$2
- new net N$48: U$5.P$16, U$6.P$1
- new net N$49: U$7.P$2, U$8.P$15
- new net N$50: U$7.P$3, U$8.P$14
- new net N$52: U$7.P$4, U$8.P$13
- new net N$53: U$7.P$5, U$8.P$12
- new net N$54: U$7.P$6, U$8.P$11
- new net N$55: U$7.P$7, U$8.P$10
- new net N$56: U$7.P$8, U$8.P$9
- new net N$57: U$7.P$9, U$8.P$8
- new net N$58: U$7.P$10, U$8.P$7
- new net N$6: SJ5.2, U$2.P$2
- new net N$61: U$7.P$11, U$8.P$6
- new net N$62: U$7.P$12, U$8.P$5
- new net N$63: U$7.P$13, U$8.P$4
- new net N$64: U$7.P$14, U$8.P$3
- new net N$65: U$7.P$15, U$8.P$2
- new net N$66: U$7.P$16, U$8.P$1
- net 8: now also PAD24.P
- net N$16: now also U$5.P$1, U$6.P$16; no longer C15.1, PAD7.P, U4.VDD3V3, U4.VDD5V
- net N$29: now also SJ7.1, SJ8.2; no longer C15.2, PAD4.P, U4.GND
- net PWR_GND: now also C16.-, C17.1, C19.-, PAD22.P, R20.1, U2.GND
- net VBAT_CUR: now also C19.+, SJ5.1, SJ6.1, SJ6.2, U2.EN, U2.IN

Commit message: Pictures and fixxes
Parts:
- removed IC5: ACS70331EOLCTR-2P5U3, ACS70331EOLCTR-2P5U3:ACS70331EOLCTR-2P5U3
- removed PAD24: (no value), wirepad:SMD2
- removed R4: 1k, SparkFun:RESISTOR0402
- added PAD23: (no value), wirepad:SMD2
- added U3: ACS70331EESATR-005B3, ACS70331EESATR-005B3:ACS70331EESATR-005B3
- R13, R14: value 10k -> 2k
Connections:
- removed net N$3: R13.1, U1.SCL
- removed net N$4: R4.2, SJ4.2
- removed net N$5: R14.1, U1.SDA
- net 0: now also R13.1, U1.SCL
- net 1: now also R14.1, U1.SDA
- net 11: now also U$3.P$7
- net 15: now also U$3.P$5
- net 16: now also U$3.P$1
- net 24: no longer U$3.P$1
- net 28: no longer U$3.P$5
- net 29: no longer U$3.P$6
- net 8: now also PAD23.P; no longer PAD24.P
- net GND: now also SJ4.2; no longer R4.1
- net MOT5_IN2: now also U$1.P$7; no longer U$1.P$6
- net PWR_GND: now also U3.GND; no longer IC5.GND
- net PWR_VCC: now also U3.VCC; no longer IC5.VCC
- net VBAT_CUR: now also U$1.P$6, U3.IP-; no longer IC5.IP-_1, IC5.IP-_2, U$1.P$7
- net VBAT_IN: now also U3.IP+; no longer IC5.IP+_1, IC5.IP+_2
- net VIN: now also U$3.P$6; no longer U$3.P$7
- net VIOUT: now also U3.VIOUT; no longer IC5.VIOUT
