File: Eagle/Maple - Clone/maplemini.sch (EAGLE design)
At the start: 32 parts, among them Q1 NPN-BJT, Q2 NPN-BJT, U1 AMS1117-3.3, X1 USB-MINIB

Commit message: reworked off proper reference boards
Parts:
- removed C10, C11: 47pF, SparkFun:CAP0402
- removed C4: 1uF, SparkFun:CAP0402
- removed Q1, Q2: NPN-BJT, SparkFun2:TRANSISTOR_NPNSOT23
- removed R10: 1.5k, SparkFun:RESISTOR0402
- removed R11: 36k, SparkFun:RESISTOR0402
- removed R2, R4: 1k, SparkFun:RESISTOR0402
- removed R3, R8: 10k, SparkFun:RESISTOR0402
- added C3: 1.0uF, SparkFun-Capacitors:1.0UF-0603-16V-10%
- added Q3, Q4: NPN-BJT, SparkFun2:TRANSISTOR_NPNSOT23
- added R13: 1.5k, SparkFun-Resistors:22OHM-0603-1/10W-1%
- added R14: 1k, SparkFun-Resistors:1KOHM-0603-1/10W-1%
- added R15: 10k, SparkFun-Resistors:10KOHM-0603-1/10W-1%
- C5, C6, C7: value 1uF -> 1.0uF; device SparkFun:CAP0402 -> SparkFun-Capacitors:1.0UF-0603-16V-10%
- D1: device SparkFun:LED1206 -> SparkFun-LED:LED0603
- R1: device SparkFun:RESISTOR0402 -> SparkFun-Resistors:1KOHM-0603-1/10W-1%
- R12: value 47k -> 39k; device SparkFun:RESISTOR0402 -> SparkFun-Resistors:39KOHM-0603-1/10W-1%
- R5: value 1k -> 51k; device SparkFun:RESISTOR0402 -> SparkFun-Resistors:47KOHM-0603-1/10W-1%
- R6, R7: device SparkFun:RESISTOR0402 -> SparkFun-Resistors:22OHM-0603-1/10W-1%
- R9: device SparkFun:RESISTOR0402 -> SparkFun-Resistors:10KOHM-0603-1/10W-1%
Connections:
- removed net AV+: C4.1, UC1.VDD_A
- removed net AV-: C4.2, UC1.VSS_A
- removed net N$1: R2.1, SJ1.2
- removed net N$4: R4.2, SJ4.2
- removed net N$51: Q2.E, R10.2
- removed net N$71: Q1.C, Q2.B, R11.2, R8.1
- removed net N$73: Q1.B, R12.1, R5.2
- new net N$3: Q3.E, R13.2
- new net N$6: Q4.B, R14.2, R5.1
- new net N$7: Q3.B, Q4.C, R12.2, R15.1
- net +5V/2: now also R15.2; no longer R8.2
- net 23_USBDP: now also R13.1; no longer C11.2, R10.1
- net 24_USBDM: no longer C10.2
- net DGND: now also C3.1, Q4.E, R12.1, SJ4.2, UC1.VSS_A; no longer C10.1, C11.1, Q1.E, R11.1, R4.1
- net DISC: now also R14.1; no longer R5.1
- net RESET: now also C3.2; no longer R3.1
- net VCC: now also Q3.C, R5.2, SJ1.2, UC1.VDD_A; no longer Q2.C, R12.2, R2.2, R3.2
Other:
- moved on the sheet: R12, R5
